Commit message: added rviz start config

File: src/robot_description/urdf/mycobot_600_urdf.urdf.xacro (robot description, xacro)
@@ -6,5 +6,5 @@
       <geometry>
 	     <!--- 0.0 0 -0.04  1.5708 3.14159-->
-       <mesh filename="package://mycobot_description/urdf/600_urdf/base.dae"/>
+       <mesh filename="package://robot_description/urdf/base.dae"/>
       </geometry>
     <origin xyz = "0 0 0 " rpy = " 0 0 0"/>
@@ -13,5 +13,5 @@
     <geometry>
 	     <!--- 0.0 0 -0.04  1.5708 3.14159-->
-       <mesh filename="package://mycobot_description/urdf/600_urdf/base.dae"/>
+       <mesh filename="package://robot_description/urdf/base.dae"/>
       </geometry>
     <origin xyz = "0 0 0 " rpy = " 0 0 0"/>
@@ -21,5 +21,5 @@
     <visual>
       <geometry>
-       <mesh filename="package://mycobot_description/urdf/600_urdf/link1.dae"/>
+       <mesh filename="package://robot_description/urdf/link1.dae"/>
       </geometry>
     <origin xyz = "0 0 0 " rpy = "0 0 3.1415926"/>
@@ -32,5 +32,5 @@
      <collision>
       <geometry>
-       <mesh filename="package://mycobot_description/urdf/600_urdf/link1.dae"/>
+       <mesh filename="package://robot_description/urdf/link1.dae"/>
       </geometry>
     <origin xyz = "0 0 0 " rpy = " 0 0 3.1415926"/>
@@ -40,5 +40,5 @@
     <visual>
       <geometry>
-       <mesh filename="package://mycobot_description/urdf/600_urdf/link2.dae"/>
+       <mesh filename="package://robot_description/urdf/link2.dae"/>
       </geometry>
     <origin xyz = "0 0 -0.080 " rpy = " 3.1415926 0 3.1415926"/>
@@ -51,5 +51,5 @@
      <collision>
      <geometry>
-       <mesh filename="package://mycobot_description/urdf/600_urdf/link2.dae"/>
+       <mesh filename="package://robot_description/urdf/link2.dae"/>
       </geometry>
     <origin xyz = "0 0 -0.080 " rpy = " 3.1415926 0 3.1415926"/>
@@ -60,5 +60,5 @@
       <geometry>
        <!--- 0.0 0 -0.04 -->
-       <mesh filename="package://mycobot_description/urdf/600_urdf/link3.dae"/>
+       <mesh filename="package://robot_description/urdf/link3.dae"/>
       </geometry>
     <origin xyz = "0 0 -0.0855 " rpy = " 3.1415926 0 3.1415926"/>
@@ -72,5 +72,5 @@
       <geometry>
        <!--- 0.0 0 -0.04 -->
-       <mesh filename="package://mycobot_description/urdf/600_urdf/link3.dae"/>
+       <mesh filename="package://robot_description/urdf/link3.dae"/>
       </geometry>
     <origin xyz = "0 0 -0.0855 " rpy = "3.1415926 0 3.1415926"/>
@@ -81,5 +81,5 @@
       <geometry>
        <!--- 0.0 0 -0.04 -->
-       <mesh filename="package://mycobot_description/urdf/600_urdf/link4.dae"/>
+       <mesh filename="package://robot_description/urdf/link4.dae"/>
       </geometry>
     <origin xyz = "0 0 0 " rpy = " 0 3.1415926 0"/>
@@ -93,5 +93,5 @@
      <geometry>
        <!--- 0.0 0 -0.04 -->
-       <mesh filename="package://mycobot_description/urdf/600_urdf/link4.dae"/>
+       <mesh filename="package://robot_description/urdf/link4.dae"/>
       </geometry>
     <origin xyz = "0 0 0 " rpy = " 0 3.1415926 0"/>
@@ -102,5 +102,5 @@
       <geometry>
        <!--- 0.0 0 -0.04 -->
-       <mesh filename="package://mycobot_description/urdf/600_urdf/link5.dae"/>
+       <mesh filename="package://robot_description/urdf/link5.dae"/>
       </geometry>
     <origin xyz = "0 0  0 " rpy = " 0  0 1.5707"/>
@@ -114,5 +114,5 @@
       <geometry>
        <!--- 0.0 0 -0.04 -->
-       <mesh filename="package://mycobot_description/urdf/600_urdf/link5.dae"/>
+       <mesh filename="package://robot_description/urdf/link5.dae"/>
       </geometry>
     <origin xyz = "0 0  0 " rpy = " 0  0 1.5707"/>
@@ -123,5 +123,5 @@
       <geometry>
        <!--- 0.0 0 -0.04 -->
-       <mesh filename="package://mycobot_description/urdf/600_urdf/link6.dae"/>
+       <mesh filename="package://robot_description/urdf/link6.dae"/>
       </geometry>
       <material name = "grey">
@@ -138,5 +138,5 @@
      <geometry>
        <!--- 0.0 0 -0.04 -->
-       <mesh filename="package://mycobot_description/urdf/600_urdf/link6.dae"/>
+       <mesh filename="package://robot_description/urdf/link6.dae"/>
       </geometry>
       <material name = "grey">
